File: hw/horrible_version/CorboIron.sch (KiCad schematic (older format))
At the start: 97 parts, among them P1 CONN_01X03, P10 CONN_01X04, P11 CONN_01X04, P2 CONN_01X03, P3 CONN_01X03, P4 Arduino_nano, P5 CONN_01X03, P6 CONN_01X04, P7 CONN_01X02, P8 CONN_01X03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

Commit message: Started pretty version
Parts:
- removed D11, D12, D13, D14: D, Diodes_SMD:DO-214BA, symbol D
- removed R24, R25, R26, R27, R28, R29, R30, R31, R32, R33, R34, R35, R36, R37, R38, R39, R40, R41, R42, R43, R44, R45, R46, R47: R, Resistors_SMD:R_1206_HandSoldering, symbol R
- removed U1, U2, U3, U4: LM324, symbol LM324
- added RV2, RV4, RV6, RV8: POT, SMD_Packages:POT_SMD, symbol POT
- added U1: 74LS08, Housings_SOIC:SOIC-14_3.9x8.7mm_Pitch1.27mm, symbol 74LS08
- added U10, U11, U12, U13, U2, U3, U4, U5, U6, U7, U8, U9: LM741, SMD_Packages:SOIC-8-N, symbol LM741
Connections:
- wire segments 332 -> 268
Other:
- moved on the sheet: P1, P2, P3, P5, Q1, Q2, Q3, Q4
