File: hw/CorboIron.sch (KiCad schematic (older format))
At the start: 97 parts, among them P1 CONN_01X03, P10 CONN_01X04, P11 CONN_01X04, P2 CONN_01X03, P3 CONN_01X03, P4 Arduino_nano, P5 CONN_01X03, P6 CONN_01X04, P7 CONN_01X02, P8 CONN_01X03, P9 CONN_01X03, Q1 IPS6041RPBF, Q2 IPS6041RPBF, Q3 IPS6041RPBF, Q4 IPS6041RPBF, U1 LM324, U14 7805, U2 LM324, U3 LM324, U4 LM324

Commit message: Completely routed but not pretty or functional, need wider traces for the heater currents!
Parts:
- D1, D11, D12, D13, D14, D3, D4, D5, D7, D9: footprint Diodes_SMD:DO-214BA -> Diodes_SMD:SOD-123
- P4: footprint (none) -> Housings_DIP:DIP-32_W15.24mm_LongPads
- R1, R10, R11, R12, R13, R14, R15, R16, R17, R18, R19, R2, R20, R21, R22, R23, R24, R25, R26, R27, R28, R29, R3, R30, R31, R32, R33, R34, R35, R36, R37, R38, R39, R4, R40, R41, R42, R43, R44, R45, R46, R47, R5, R6, R7, R8, R9: footprint Resistors_SMD:R_1206_HandSoldering -> Resistors_SMD:R_0805
- U1, U2, U3, U4: footprint (none) -> SMD_Packages:SO14N
Connections:
- wire segments 332 -> 300

Commit message: Added pulldown resistors for opamp logic started placeing refdes and values on silkscreen
Parts:
- added R48, R49, R50, R51: 27K, Resistors_SMD:R_0805, symbol R
- C1, C4, C5, C6: value CP1 -> 1uF
- C10, C7: value CP1 -> 100u
- C2: value CP1 -> 4u7
- C3: value CP1 -> 220u
- C8, C9: value C -> 10n
- R1, R13, R17, R18, R19, R20, R21, R22, R23, R5, R9: value R -> 100K
- R10, R14, R2, R6: value R -> 680K
- R11, R15, R34, R35, R40, R41, R46, R47, R7: value R -> 4K7
- R12, R16, R4, R8: value R -> 1K
- R24, R30, R36, R42: value R -> 22K
- R25, R31, R37, R43: value R -> 6K8
- R26, R32, R38, R44: value R -> 150K
- R27, R33, R39, R45: value R -> 2K7
- R28, R29, R3: value R -> 4k7
- RV1, RV3, RV5, RV7: value POT -> 5K
Connections:
- wire segments 300 -> 312
Other:
- note added: "High value current limiting resistor because negative supply rail is low current"
- note added: "OVER HEAT 1"
- note added: "OVER HEAT 2"
- note added: "OVER HEAT 3"

Commit message: Checked footprints, design should be ready for production
Connections:
- wire segments 312 -> 309
Changed lines of the file:
@@
 TEMP0_OK
-$Comp
-L GND #PWR013
-U 1 1 56EDAFF5
-P 13950 8200
-F 0 "#PWR013" H 13950 7950 50  0001 C CNN
-F 1 "GND" H 13950 8050 50  0000 C CNN
-F 2 "" H 13950 8200 50  0000 C CNN
-F 3 "" H 13950 8200 50  0000 C CNN
-	1    13950 8200
-	1    0    0    -1
-$EndComp
 $Comp
 L GND #PWR014
@@
 TEMP1_OK
 $Comp
-L GND #PWR028
-U 1 1 56EE796D
-P 13950 6300
-F 0 "#PWR028" H 13950 6050 50  0001 C CNN
-F 1 "GND" H 13950 6150 50  0000 C CNN
-F 2 "" H 13950 6300 50  0000 C CNN
-F 3 "" H 13950 6300 50  0000 C CNN
-	1    13950 6300
-	1    0    0    -1
-$EndComp
-$Comp
 L GND #PWR029
 U 1 1 56EE7975
@@
 Text Label 10700 2300 0    60   ~ 0
 TEMP3_OK
-$Comp
-L GND #PWR054
-U 1 1 56EE7FE7
-P 13950 2400
-F 0 "#PWR054" H 13950 2150 50  0001 C CNN
-F 1 "GND" H 13950 2250 50  0000 C CNN
-F 2 "" H 13950 2400 50  0000 C CNN
-F 3 "" H 13950 2400 50  0000 C CNN
-	1    13950 2400
-	1    0    0    -1
-$EndComp
 $Comp
 L GND #PWR055
@@
 	10700 8100 11100 8100
 Wire Wire Line
-	13950 8200 14050 8200
-Wire Wire Line
 	12300 8000 13050 8000
 Wire Wire Line
@@
 	10700 6200 11100 6200
 Wire Wire Line
-	13950 6300 14050 6300
-Wire Wire Line
 	12300 6100 13050 6100
 Wire Wire Line
@@
 	10700 2300 11100 2300
 Wire Wire Line
-	13950 2400 14050 2400
-Wire Wire Line
 	12300 2200 13050 2200

Commit message: dont remember exactly :)
Parts:
- removed R48, R49, R50, R51: 27K, Resistors_SMD:R_0805, symbol R
- C1, C4, C5, C6: value 1uF -> CP1
- C10, C7: value 100u -> CP1
- C2: value 4u7 -> CP1
- C3: value 220u -> CP1
- C8, C9: value 10n -> C
- R1, R13, R17, R18, R19, R20, R21, R22, R23, R5, R9: value 100K -> R
- R10, R14, R2, R6: value 680K -> R
- R11, R15, R34, R35, R40, R41, R46, R47, R7: value 4K7 -> R
- R12, R16, R4, R8: value 1K -> R
- R24, R30, R36, R42: value 22K -> R
- R25, R31, R37, R43: value 6K8 -> R
- R26, R32, R38, R44: value 150K -> R
- R27, R33, R39, R45: value 2K7 -> R
- R28, R29, R3: value 4k7 -> R
- RV1, RV3, RV5, RV7: value 5K -> POT
Connections:
- wire segments 309 -> 300
Other:
- note removed: "High value current limiting resistor because negative supply rail is low current"
- note removed: "OVER HEAT 1"
- note removed: "OVER HEAT 2"
- note removed: "OVER HEAT 3"

Commit message: Reverted schematic
Parts:
- added R48, R49, R50, R51: 27K, Resistors_SMD:R_0805, symbol R
- C1, C4, C5, C6: value CP1 -> 1uF
- C10, C7: value CP1 -> 100u
- C2: value CP1 -> 4u7
- C3: value CP1 -> 220u
- C8, C9: value C -> 10n
- R1, R13, R17, R18, R19, R20, R21, R22, R23, R5, R9: value R -> 100K
- R10, R14, R2, R6: value R -> 680K
- R11, R15, R34, R35, R40, R41, R46, R47, R7: value R -> 4K7
- R12, R16, R4, R8: value R -> 1K
- R24, R30, R36, R42: value R -> 22K
- R25, R31, R37, R43: value R -> 6K8
- R26, R32, R38, R44: value R -> 150K
- R27, R33, R39, R45: value R -> 2K7
- R28, R29, R3: value R -> 4k7
- RV1, RV3, RV5, RV7: value POT -> 5K
Connections:
- wire segments 300 -> 309
Other:
- note added: "High value current limiting resistor because negative supply rail is low current"
- note added: "OVER HEAT 1"
- note added: "OVER HEAT 2"
- note added: "OVER HEAT 3"
